File: pcb/main/kicad_project/PCB_FujitoraBot2.kicad_sch (KiCad schematic)
At the start: 99 parts, among them IC1 AS5040, IC2 AS5040, J1 MORRO1, SW2 SW_Reset, SW4 SW_Push, U2 LM1117MP-3.3, U3 MPU-6500, Y1 Crystal

Commit message: Finaliza el ruteo de la PCB_main a falta de los encoders
Parts:
- removed Y1: Crystal, Crystal:Crystal_SMD_3225-4Pin_3.2x2.5mm, symbol Device:Crystal
- added Y1: Crystal_GND24, Crystal:Crystal_SMD_TXC_7M-4Pin_3.2x2.5mm, symbol Device:Crystal_GND24
- DC-DC1: footprint custom_footprints:SOP8 -> custom_footprints:SOP8_with_gnd_pad
- U3: footprint Sensor_Motion:InvenSense_QFN-24_3x3mm_P0.4mm -> custom_footprints:FujitoraBot2_giro_MPU6500
Connections:
- net +3V3: no longer USB1.11 (VBUS), USB1.2 (VBUS)
- net GND: now also Y1.2, Y1.4
- net at C26.2, DEIXAME_QUE_PENSE_1.6 (PH1/OSC_OUT): now also Y1.1
- net at C25.2, DEIXAME_QUE_PENSE_1.5 (PH0/OSC_IN): now also Y1.3
- no-connect marks 37 -> 39
Other:
- moved on the sheet: C25, C26
